File: eletronica/ponta-de-prova-logica/ppl-01/fontes-kicad/ppl-01.kicad_pcb (KiCad board)
At the start: 2 copper layers, 49.5 x 45.7 mm, 57 parts, among them J1 Conn_01x02, Q1 BC847, SW1 SW_DPDT_x2, SW2 SW_DPDT_x2, U1 LM339

Commit message: Projeto Ponta de Prova Lógica - Modelo PPL-01 preparado conforme orientações do guia da licença CERN-OHL-S v2 e pronto para liberação.
Parts:
- added R***: QR_CODE_URL_Fontes_PPL-01, contornos-personalizados:QR_CODE_URL_Fontes_PPL-01, F.Cu at (148.6, 115.1)
- moved G*** 4.19 mm to (144.4, 115.1)
Other:
- board text added: "Fontes"
- board text added: "Licended under CERN-OHL-S v2"
- board text removed: "........................"
